File: aero-dev/aero-dev.kicad_sch (KiCad schematic)
At the start: 32 parts, among them J1 Conn_01x03_Pin, J2 USB_C_Receptacle_USB2.0_16P, J3 Conn_ARM_SWD_TagConnect_TC203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, J4 Conn_01x03_Pin, J5 Conn_01x03_Pin, J6 Conn_01x03_Pin, J7 Barrel_Jack_Switch, U4 SRV05-4, U5 STM32F103C8Tx, U6 AMS1117-3.3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

Commit message: Finalize production files and minor edits
Parts:
- C21: footprint Capacitor_SMD:C_0603_1608Metric -> Capacitor_SMD:C_0805_2012Metric
- J1, J4, J5, J6: now not fitted
- LED1: LCSC (none) -> C2986059
Changed lines of the file:
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@@
+			)
+		)
+		(property "LCSC" "C2986059"
+			(at 248.92 143.51 90)
+			(effects
+				(font
+					(size 1.27 1.27)
+				)
+				(hide yes)
 			)
 		)
@@
 		(in_bom yes)
 		(on_board yes)
-		(dnp no)
+		(dnp yes)
 		(fields_autoplaced yes)
 		(property "Reference" "J4"
@@
 			)
 		)
-		(property "Footprint" "Capacitor_SMD:C_0603_1608Metric"
+		(property "Footprint" "Capacitor_SMD:C_0805_2012Metric"
 			(at 72.0852 35.56 0)
 			(effects
@@
 		(in_bom yes)
 		(on_board yes)
-		(dnp no)
+		(dnp yes)
 		(fields_autoplaced yes)
 		(property "Reference" "J6"
@@
 		(in_bom yes)
 		(on_board yes)
-		(dnp no)
+		(dnp yes)
 		(fields_autoplaced yes)
 		(property "Reference" "J1"
@@
 		(in_bom yes)
 		(on_board yes)
-		(dnp no)
+		(dnp yes)
 		(fields_autoplaced yes)
 		(property "Reference" "J5"
