File: aero-dev/regulator.kicad_sch (KiCad schematic)
At the start: 13 parts, among them U1 TPS5450DDAR

Commit message: Finalize production files and minor edits
Parts:
- LED2: LCSC (none) -> C2986058
- U1: LCSC (none) -> C114425
Changed lines of the file:
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@@
+			)
+		)
+		(property "LCSC" "C114425"
+			(at 68.58 53.34 0)
+			(effects
+				(font
+					(size 1.27 1.27)
+				)
+				(hide yes)
 			)
 		)
@@
 			(effects
 				(font
+					(size 1.27 1.27)
+				)
+				(hide yes)
+			)
+		)
+		(property "LCSC" "C2986058"
+			(at 152.4 72.39 90)
+			(effects
+				(font
